File: isp32/isp32.kicad_pcb (KiCad board)
At the start: 2 copper layers, 53 x 48 mm, 121 parts, among them J1 BAT1, J10 LoRa_ANT, J11 Power Modules, J12 Micro_SD_Card, J2 Switching, J3 USB_C_Receptacle_USB2.0, J4 ADC, J5 GPS_ANT, J6 F0, J7 F1, J8 BUZZ, J9 ANT, M1 Motor_Servo, M2 Motor_Servo, M3 Motor_Servo, M4 Motor_Servo, Q1 BSS138, Q2 S8050, Q3 IRLML6402, Q4 BSS138, Q5 IRLML6402, Q6 IRLML6402, Q8 BSS138, Q9 BSS138, SW1 RST, U1 AZ1117-3.3, U10 BMP280, U11 MPU-9250, U2 MP2315, U3 STM32G030F6, U4 AZ1117-1.8, U6 24LC32, U7 NEO-XM, U8 ESP32-S3-WROOM-1U, U9 RFM98W-315S2

Commit message: feat: isp32 fix bugs
Parts:
- removed C1, C18, C8: 22u, Capacitor_SMD:C_0603_1608Metric
- removed C2: 220u, Capacitor_Tantalum_SMD:CP_EIA-3528-12_Kemet-T
- removed C24, C4: 100n, Capacitor_SMD:C_0603_1608Metric
- removed C7: NC, Capacitor_SMD:C_0603_1608Metric
- removed J8: BUZZ, Connector_PinHeader_1.27mm:PinHeader_1x02_P1.27mm_Vertical
- removed JP1: MPU VIO, Jumper:SolderJumper-3_P1.3mm_Bridged12_RoundedPad1.0x1.5mm_NumberLabels
- removed L3: 5.5, Inductor_SMD:L_Sunlord_SWPA5020S
- removed Q8, Q9: BSS138, Package_TO_SOT_SMD:SOT-23
- removed R10: 7k5, Resistor_SMD:R_0603_1608Metric
- removed R11: 40.2k, Resistor_SMD:R_0603_1608Metric
- removed R13, R17, R28, R29: 10k, Resistor_SMD:R_0603_1608Metric
- removed R21: 75k, Resistor_SMD:R_0603_1608Metric
- removed R3: 100k, Resistor_SMD:R_0603_1608Metric
- removed R8: 20, Resistor_SMD:R_0603_1608Metric
- removed R9: 20k, Resistor_SMD:R_0603_1608Metric
- removed U11: MPU-9250, Sensor_Motion:InvenSense_QFN-24_3x3mm_P0.4mm
- removed kibuzzard-642D96EE: G***, kibuzzard-642D96EE
- removed kibuzzard-642D96F8: G***, kibuzzard-642D96F8
- added J13: VIN_SELECT, Connector_PinHeader_2.54mm:PinHeader_1x03_P2.54mm_Vertical, F.Cu at (90.7, 59.9)
- added J14: BUZZ, Connector_Molex:Molex_PicoBlade_53261-0271_1x02-1MP_P1.25mm_Horizontal, F.Cu at (90.4, 74.0)
- added kibuzzard-661FABB5: G***, kibuzzard-661FABB5, B.Cu at (115.9, 36.1)
- added kibuzzard-661FAECF: G***, kibuzzard-661FAECF, F.Cu at (119.9, 58.4)
- added kibuzzard-661FBC0A: G***, kibuzzard-661FBC0A, F.Cu at (92.7, 63.9)
- added kibuzzard-661FBC21: G***, kibuzzard-661FBC21, F.Cu at (92.7, 61.2)
- C22: value 10n -> 1u
- C5: moved to F.Cu
- J1: footprint Connector_AMASS:AMASS_XT60-M_1x02_P7.20mm_Vertical -> Connector_JST:JST_XH_S2B-XH-A-1_1x02_P2.50mm_Horizontal
- J11, Q6, R26: moved to B.Cu
- J12: footprint Connector_Card:microSD_HC_Molex_47219-2001 -> Connector_Card:microSD_HC_Wuerth_693072010801
- J2: value Switching -> ExtBoard
- R22, R25: value 10k -> 1k
- U2: value MP2315 -> BA05C; footprint Package_TO_SOT_SMD:TSOT-23-8 -> Package_TO_SOT_SMD:TO-252-2
- U4: value AZ1117-1.8 -> LSM6DSM; footprint Package_TO_SOT_SMD:SOT-89-3 -> Package_LGA:LGA-14_3x2.5mm_P0.5mm_LayoutBorder3x4y
- moved kibuzzard-641A7704 46.4 mm to (87.8, 71.5)
- moved R2 26.6 mm to (107.0, 54.8), turned to 0 degrees
- moved U4 21.0 mm to (89.4, 38.2)
- moved D1 18.6 mm to (78.2, 63.7), turned to 90 degrees
- moved Q6 17.9 mm to (78.5, 58.7), turned to 180 degrees
- moved R26 15.5 mm to (80.5, 62.8), turned to -90 degrees
- moved D6 10.1 mm to (87.3, 63.2)
- moved C23 8.66 mm to (86.7, 38.1)
- moved J1 7.93 mm to (83.8, 61.0), turned to -90 degrees
- moved C5 7.16 mm to (87.1, 62.6), turned to -90 degrees
- moved J11 5.25 mm to (83.1, 68.8), turned to -90 degrees
- moved D2 3.28 mm to (113.1, 72.8), turned to 90 degrees
- moved C12 3.24 mm to (103.8, 59.8)
- moved D4 3.21 mm to (104.2, 72.8), turned to 90 degrees
- moved R25 3.11 mm to (104.2, 69.7), turned to 90 degrees
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Connections:
- D6 pad 2: Net-(D6-Pad2) -> Net-(D6-A2)
- D8 pad 2: Net-(C1-Pad1) -> Net-(D8-A)
- J1 pad 1: GND -> Net-(D6-A2)
- J1 pad 2: Net-(D6-Pad2) -> GND
- J11 pad 1: +BATT -> Net-(D8-A)
- J11 pad 2: +BATT -> GND
- J11 pad 3: GND -> Net-(J11-Pin_3)
- J11 pad 4: Net-(C1-Pad1) -> Net-(J11-Pin_3)
- J6 pad 1: Net-(J6-Pad1) -> Net-(J6-Pin_1)
- J7 pad 1: Net-(J7-Pad1) -> Net-(J7-Pin_1)
- Q3 pad 3: Net-(J6-Pad1) -> Net-(J6-Pin_1)
- Q5 pad 3: Net-(J7-Pad1) -> Net-(J7-Pin_1)
- Q6 pad 3: Net-(D6-Pad2) -> Net-(D6-A2)
- R22 pad 2: Net-(J6-Pad1) -> FIRE0
- R25 pad 2: Net-(J7-Pad1) -> FIRE1
- U2 pad 2: +BATT -> GND
- U2 pad 3: Net-(C4-Pad2) -> Net-(D8-A)
- U4 pad 1: GND -> unconnected-(U4-SDO/SA0-Pad1)
- U4 pad 2: +1V8 -> GND
- U4 pad 3: +3V3 -> GND
Routing:
- net Net-(C1-Pad1): track 67.4 -> 0.00 mm, vias 3 -> 0
- net +1V8: track 48.8 -> 0.00 mm, vias 4 -> 0
- net Net-(J14-Pin_2): track 69.9 -> 25.8 mm, vias 0 -> 1
- net MPU_VIO_SEL: track 41.5 -> 0.00 mm, vias 2 -> 0
- net IO0: track 44.2 -> 2.82 mm
- net GND: track 43.3 -> 4.23 mm, vias 94 -> 65
- net SCL: track 75.7 -> 111.7 mm, vias 5 -> 4
- net Net-(D6-Pad2): track 24.2 -> 0.00 mm
- net RGB: track 86.0 -> 63.9 mm
- net Net-(Q8-Pad2): track 21.6 -> 0.00 mm
- net Net-(Q9-Pad2): track 21.6 -> 0.00 mm, vias 2 -> 0
- net TX1: track 47.8 -> 27.9 mm, vias 8 -> 0
- net Net-(D8-A): track 0.00 -> 18.9 mm, vias 0 -> 1
- net +3V3: track 211.1 -> 228.1 mm, vias 12 -> 11
- net EXT_INT: track 44.8 -> 59.9 mm, vias 2 -> 8
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Other:
- board text added: "+ + - OUT"
- board text added: "3V3 GND INT SCL SDA"
- board text added: "BSD-3-Clause open source hardware By @wilicw Rev. 2024.16"
- board text added: "NCKU ISP Avionics ISP32 v3.0"
- board text removed: "BSD-3-Clause open source hardware By @wilicw"
- board text removed: "NCKU ISP Avionics ISP32 v2.1"
- board text removed: "VCC GND INT SCL SDA"

Commit message: feat: re-design schematics
Parts:
- removed R30, R33: 10k, Resistor_SMD:R_0603_1608Metric
- added D9: D_Small, Diode_SMD:D_SOD-123, F.Cu at (84.3, 74.0)
- added R3: 100, Resistor_SMD:R_0603_1608Metric, B.Cu at (98.8, 49.4)
- J9: moved to B.Cu
- R2: moved to F.Cu
- moved kibuzzard-661FAECF 8.38 mm to (125.6, 64.5), turned to 90 degrees
- moved R1 7.85 mm to (78.5, 40.9)
- moved J9 4.77 mm to (127.2, 54.9)
- moved R2 4.14 mm to (111.0, 53.7), turned to 180 degrees
- moved U9 2.47 mm to (114.6, 63.2)
- moved kibuzzard-642D97EE 1.86 mm to (126.3, 64.4)
- moved D3 1.56 mm to (82.5, 36.8)
- moved kibuzzard-641A73E5 1.56 mm to (79.1, 36.7)
- moved D5 1.56 mm to (82.5, 38.9)
- moved R18 1.56 mm to (85.6, 39.0)
- moved R19 1.56 mm to (85.6, 36.8)
- moved kibuzzard-641A73FA 1.56 mm to (78.7, 38.9)
- moved U8 0.16 mm to (99.0, 44.0)
Connections:
- J12 pad 1: unconnected-(J12-DAT2-Pad1) -> SD_D2
- J12 pad 2: SD_SS -> SD_D3
- J12 pad 3: MOSI_2 -> SD_CMD
- J12 pad 5: SCK_2 -> SD_CLK
- J12 pad 7: MISO_2 -> SD_D0
- J12 pad 8: unconnected-(J12-DAT1-Pad8) -> SD_D1
- Q2 pad 1: Buzz -> Net-(Q2-B)
- U8 pad 18: unconnected-(U8-IO10-Pad18) -> SD_D3
- U8 pad 19: unconnected-(U8-IO11-Pad19) -> SD_CMD
- U8 pad 20: unconnected-(U8-IO12-Pad20) -> SD_CLK
- U8 pad 21: unconnected-(U8-IO13-Pad21) -> SD_D0
- U8 pad 22: unconnected-(U8-IO14-Pad22) -> SD_D1
- U8 pad 23: LORA_RST -> LORA_SS
- U8 pad 31: LORA_BUSY -> unconnected-(U8-IO38-Pad31)
- U8 pad 32: MOSI_2 -> LORA_D1
- U8 pad 33: SCK_2 -> LORA_BUSY
- U8 pad 34: MISO_2 -> LORA_RST
- U8 pad 38: LORA_SS -> unconnected-(U8-IO2-Pad38)
- U8 pad 5: SD_SS -> unconnected-(U8-IO5-Pad5)
- U8 pad 7: unconnected-(U8-IO7-Pad7) -> SD_D2
- U9 pad 15: unconnected-(U9-DIO1-Pad15) -> LORA_D1
Routing:
- net +3V3: track 228.1 -> 35.8 mm, vias 11 -> 2
- net +5V: track 141.7 -> 0.00 mm
- net SCL: track 111.7 -> 0.00 mm, vias 4 -> 0
- net SDA: track 102.5 -> 0.00 mm, vias 4 -> 0
- net +BATT: track 78.8 -> 0.00 mm, vias 2 -> 0
- net RGB: track 63.9 -> 0.00 mm, vias 5 -> 0
- net EXT_INT: track 59.9 -> 0.00 mm, vias 8 -> 0
- net RX1: track 40.7 -> 0.00 mm, vias 2 -> 0
- net FIRE0: track 33.9 -> 0.00 mm
- net LORA_BUSY: track 30.6 -> 0.00 mm, vias 1 -> 0
- net LORA_SS: track 30.4 -> 0.00 mm, vias 1 -> 0
- net TX1: track 27.9 -> 0.00 mm
- net MISO_2: track 27.4 -> 0.00 mm, vias 1 -> 0
- net SCK_2: track 26.4 -> 0.00 mm, vias 1 -> 0
- net Net-(D9-A): track 25.8 -> 0.00 mm, vias 1 -> 0
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
Commit message: chore: update isp32 project files
Parts:
- added TP2: TP-3V3, TestPoint:TestPoint_Pad_D1.0mm, F.Cu at (104.0, 55.8)
- added kibuzzard-66439A83: G***, kibuzzard-66439A83, B.Cu at (92.2, 42.0)
- added kibuzzard-66439ACD: G***, kibuzzard-66439ACD, B.Cu at (89.2, 35.8)
- added kibuzzard-66439AF0: G***, kibuzzard-66439AF0, B.Cu at (119.8, 72.4)
- added kibuzzard-66439B33: G***, kibuzzard-66439B33, F.Cu at (114.0, 35.2)
- added kibuzzard-66439B8F: G***, kibuzzard-66439B8F, F.Cu at (101.4, 70.2)
- added kibuzzard-66439C31: G***, kibuzzard-66439C31, F.Cu at (101.6, 55.8)
- R22, R25: value 1k -> 10k
- moved R15 2.44 mm to (104.3, 63.9)
Connections:
- R22 pad 2: FIRE0 -> Net-(J6-Pin_1)
- R25 pad 2: FIRE1 -> Net-(J7-Pin_1)
Routing:
- net +3V3: track 35.8 -> 213.4 mm, vias 2 -> 10
- net +5V: track 0.00 -> 130.2 mm, vias 0 -> 1
- net SCL: track 0.00 -> 88.2 mm, vias 0 -> 4
- net SDA: track 0.00 -> 83.2 mm, vias 0 -> 1
- net +BATT: track 0.00 -> 80.6 mm, vias 0 -> 2
- net RGB: track 0.00 -> 48.9 mm, vias 0 -> 5
- net EXT_INT: track 0.00 -> 46.4 mm, vias 0 -> 2
- net Net-(D9-A): track 0.00 -> 43.4 mm, vias 0 -> 1
- net LORA_BUSY: track 0.00 -> 33.4 mm, vias 0 -> 1
- net LORA_D1: track 0.00 -> 33.1 mm, vias 0 -> 1
- net RX1: track 0.00 -> 27.7 mm, vias 0 -> 2
- net FIRE1: track 0.00 -> 26.0 mm, vias 0 -> 2
- net MISO_1: track 0.00 -> 25.2 mm, vias 0 -> 1
- net FIRE0: track 0.00 -> 24.1 mm
- net INDI: track 0.00 -> 22.9 mm
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