File: isp32/isp32.kicad_sch (KiCad schematic)
At the start: 105 parts, among them J1 BAT1, J10 LoRa_ANT, J11 Power Modules, J12 Micro_SD_Card, J2 Switching, J3 USB_C_Receptacle_USB2.0, J4 ADC, J5 GPS_ANT, J6 F0, J7 F1, J8 BUZZ, J9 ANT, M1 Motor_Servo, M2 Motor_Servo, M3 Motor_Servo, M4 Motor_Servo, Q1 BSS138, Q2 S8050, Q3 IRLML6402, Q4 BSS138, Q5 IRLML6402, Q6 IRLML6402, Q8 BSS138, Q9 BSS138, SW1 RST, U1 AZ1117-3.3, U10 BMP280, U11 MPU-9250, U2 MP2315, U3 STM32G030F6, U4 AZ1117-1.8, U6 24LC32, U7 NEO-XM, U8 ESP32-S3-WROOM-1U, U9 RFM98W-315S2

Commit message: feat: isp32 fix bugs
Parts:
- removed C1, C18, C8: 22u, Capacitor_SMD:C_0603_1608Metric, symbol Device:C_Small
- removed C2: 220u, Capacitor_Tantalum_SMD:CP_EIA-3528-12_Kemet-T, symbol Device:C_Small
- removed C24, C4: 100n, Capacitor_SMD:C_0603_1608Metric, symbol Device:C_Small
- removed C7: NC, Capacitor_SMD:C_0603_1608Metric, symbol Device:C_Small
- removed J8: BUZZ, Connector_PinHeader_1.27mm:PinHeader_1x02_P1.27mm_Vertical, symbol Connector_Generic:Conn_01x02
- removed JP1: MPU VIO, Jumper:SolderJumper-3_P1.3mm_Bridged12_RoundedPad1.0x1.5mm_NumberLabels, symbol Jumper:SolderJumper_3_Bridged12
- removed L3: 5.5, Inductor_SMD:L_Sunlord_SWPA5020S, symbol Device:L_Small
- removed Q8, Q9: BSS138, Package_TO_SOT_SMD:SOT-23, symbol Transistor_FET:BSS138
- removed R10: 7k5, Resistor_SMD:R_0603_1608Metric, symbol Device:R_Small
- removed R11: 40.2k, Resistor_SMD:R_0603_1608Metric, symbol Device:R_Small
- removed R13, R17, R28, R29: 10k, Resistor_SMD:R_0603_1608Metric, symbol Device:R_Small
- removed R21: 75k, Resistor_SMD:R_0603_1608Metric, symbol Device:R_Small
- removed R3: 100k, Resistor_SMD:R_0603_1608Metric, symbol Device:R_Small
- removed R8: 20, Resistor_SMD:R_0603_1608Metric, symbol Device:R_Small
- removed R9: 20k, Resistor_SMD:R_0603_1608Metric, symbol Device:R_Small
- removed U11: MPU-9250, Sensor_Motion:InvenSense_QFN-24_3x3mm_P0.4mm, symbol Sensor_Motion:MPU-9250
- removed U2: MP2315, Package_TO_SOT_SMD:TSOT-23-8, symbol MP2315:MP2315
- removed U4: AZ1117-1.8, Package_TO_SOT_SMD:SOT-89-3, symbol Regulator_Linear:AZ1117-1.8
- added J13: VIN_SELECT, Connector_PinHeader_2.54mm:PinHeader_1x03_P2.54mm_Vertical, symbol Connector_Generic:Conn_01x03
- added J14: BUZZ, Connector_Molex:Molex_PicoBlade_53261-0271_1x02-1MP_P1.25mm_Horizontal, symbol Connector_Generic_MountingPin:Conn_01x02_MountingPin
- added U2: BA05C, Package_TO_SOT_SMD:TO-252-2, symbol Regulator_Linear:AP2204R-5.0
- added U4: LSM6DSM, Package_LGA:LGA-14_3x2.5mm_P0.5mm_LayoutBorder3x4y, symbol Sensor_Motion:LSM6DSM
- C22: value 10n -> 1u
- J1: footprint Connector_AMASS:AMASS_XT60-M_1x02_P7.20mm_Vertical -> Connector_JST:JST_XH_S2B-XH-A-1_1x02_P2.50mm_Horizontal
- J12: footprint Connector_Card:microSD_HC_Molex_47219-2001 -> Connector_Card:microSD_HC_Wuerth_693072010801
- J2: value Switching -> ExtBoard
- R22, R25: value 10k -> 1k
Connections:
- net +3V3: now also U4.12 (CS), U4.5 (VDDIO), U4.8 (VDD)
- net +5V: now also J14.1 (Pin_1)
- net +BATT: now also J13.2 (Pin_2); no longer J11.1 (Pin_1), J11.2 (Pin_2)
- net FIRE0: now also R22.2
- net FIRE1: now also R25.2
- net GND: now also J1.2 (Pin_2), J11.2 (Pin_2), J14.MP (MountPin), U2.2 (GND), U4.2 (SDX), U4.3 (SCX), U4.6 (GND), U4.7 (GND); no longer J1.1 (Pin_1), J11.3 (Pin_3)
- net IMU_INT: now also U4.4 (INT1)
- net SCL: now also U4.13 (SCL)
- net SDA: now also U4.14 (SDA)
- net at D8.2 (A): now also J11.1 (Pin_1), U2.3 (VOUT); no longer J11.4 (Pin_4)
- net at LS1.N, Q2.2 (C): now also J14.2 (Pin_2)
- net at J6.1 (Pin_1), Q3.3 (D): no longer R22.2
- net at D6.2 (A2), Q6.3 (D): now also J1.1 (Pin_1); no longer J1.2 (Pin_2)
- net at J7.1 (Pin_1), Q5.3 (D): no longer R25.2
- new net: J11.3 (Pin_3), J11.4 (Pin_4), J13.3 (Pin_3)
- new net: J13.1 (Pin_1), U2.1 (VIN)
- no-connect marks 38 -> 39
Other:
- moved on the sheet: D7, D8, J1, J11

Commit message: feat: re-design schematics
Parts:
- removed R30, R33: 10k, Resistor_SMD:R_0603_1608Metric, symbol Device:R_Small
- added D9: D_Small, Diode_SMD:D_SOD-123, symbol Device:D_Small
- added R3: 100, Resistor_SMD:R_0603_1608Metric, symbol Device:R_Small
Connections:
- net +5V: now also D9.1 (K)
- net Buzz: now also R3.1; no longer Q2.1 (B)
- net LORA_BUSY: now also U8.33 (IO40); no longer U8.31 (IO38)
- net LORA_RST: now also U8.34 (IO41); no longer U8.23 (IO21)
- net LORA_SS: now also U8.23 (IO21); no longer U8.38 (IO2)
- net LORA_D1: now reaches U9.15 (DIO1)
- net LORA_D1: now also U8.32 (IO39)
- net SD_D3: now reaches U8.18 (IO10)
- net SD_D3: now also J12.2 (DAT3/CD)
- net SD_CMD: now reaches U8.19 (IO11)
- net SD_CMD: now also J12.3 (CMD)
- net SD_CLK: now reaches U8.20 (IO12)
- net SD_CLK: now also J12.5 (CLK)
- net SD_D0: now reaches U8.21 (IO13)
- net SD_D0: now also J12.7 (DAT0)
- net SD_D1: now reaches U8.22 (IO14)
- net SD_D1: now also J12.8 (DAT1)
- net SD_D2: now reaches U8.7 (IO7)
- net SD_D2: now also J12.1 (DAT2)
- net at J14.2 (Pin_2), LS1.N, Q2.2 (C): now also D9.2 (A)
- removed net MISO_2: J12.7 (DAT0), U8.34 (IO41)
- removed net MOSI_2: J12.3 (CMD), U8.32 (IO39)
- removed net SCK_2: J12.5 (CLK), U8.33 (IO40)
- net SD_SS: no longer names the net of U8.5 (IO5)
- net SD_SS: no longer J12.2 (DAT3/CD)
- new net: Q2.1 (B), R3.2
- no-connect marks 39 -> 34
Other:
- moved on the sheet: LS1

Commit message: chore: update isp32 project files
Parts:
- added TP2: TP-3V3, TestPoint:TestPoint_Pad_D1.0mm, symbol Connector:TestPoint
- R22, R25: value 1k -> 10k
Connections:
- net +3V3: now also TP2.1
- net FIRE0: no longer R22.2
- net FIRE1: no longer R25.2
- net at J6.1 (Pin_1), Q3.3 (D): now also R22.2
- net at J7.1 (Pin_1), Q5.3 (D): now also R25.2
Changed lines of the file:
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@@
   (junction (at 31.115 146.05) (diameter 0) (color 0 0 0 0)
   )
-  (junction (at 331.47 40.005) (diameter 0) (color 0 0 0 0)
-  )
   (junction (at 329.565 118.11) (diameter 0) (color 0 0 0 0)
   )
@@
   (junction (at 159.385 130.81) (diameter 0) (color 0 0 0 0)
   )
+  (junction (at 350.52 45.085) (diameter 0) (color 0 0 0 0)
+  )
   (junction (at 151.765 135.89) (diameter 0) (color 0 0 0 0)
   )
@@
   (junction (at 331.47 29.845) (diameter 0) (color 0 0 0 0)
   )
+  (junction (at 305.435 45.72) (diameter 0) (color 0 0 0 0)
+  )
   (junction (at 350.52 59.055) (diameter 0) (color 0 0 0 0)
   )
@@
   (junction (at 180.975 166.37) (diameter 0) (color 0 0 0 0)
   )
-  (junction (at 286.385 40.64) (diameter 0) (color 0 0 0 0)
-  )
   (junction (at 305.435 30.48) (diameter 0) (color 0 0 0 0)
   )
@@
     (stroke (width 0) (type default))
   )
-  (wire (pts (xy 331.47 45.085) (xy 345.44 45.085))
-    (stroke (width 0) (type default))
-  )
   (wire (pts (xy 116.205 88.9) (xy 127.635 88.9))
     (stroke (width 0) (type default))
@@
     (stroke (width 0) (type dash))
   )
-  (wire (pts (xy 286.385 45.72) (xy 286.385 40.64))
-    (stroke (width 0) (type default))
-  )
   (wire (pts (xy 68.58 90.17) (xy 63.5 90.17))
     (stroke (width 0) (type default))
@@
     (stroke (width 0) (type dash))
   )
-  (wire (pts (xy 331.47 45.085) (xy 331.47 40.005))
-    (stroke (width 0) (type default))
-  )
   (wire (pts (xy 331.47 29.845) (xy 331.47 32.385))
     (stroke (width 0) (type default))
@@
     (stroke (width 0) (type dash))
   )
+  (wire (pts (xy 345.44 45.085) (xy 350.52 45.085))
+    (stroke (width 0) (type default))
+  )
   (wire (pts (xy 139.065 81.28) (xy 135.255 81.28))
     (stroke (width 0) (type default))
@@
     (stroke (width 0) (type dash))
   )
+  (wire (pts (xy 147.955 81.28) (xy 153.67 81.28))
+    (stroke (width 0) (type default))
+  )
   (polyline (pts (xy 24.638 104.14) (xy 206.248 104.14))
     (stroke (width 0) (type dash))
@@
     (stroke (width 0) (type dash))
   )
-  (wire (pts (xy 286.385 45.72) (xy 300.355 45.72))
-    (stroke (width 0) (type default))
-  )
   (polyline (pts (xy 211.455 66.675) (xy 270.51 66.675))
     (stroke (width 0) (type dash))
@@
     (stroke (width 0) (type dash))
   )
+  (wire (pts (xy 300.355 45.72) (xy 305.435 45.72))
+    (stroke (width 0) (type default))
+  )
   (polyline (pts (xy 270.51 109.22) (xy 270.51 199.39))
     (stroke (width 0) (type dash))
@@
     )
   )
+  (symbol (lib_id "Connector:TestPoint") (at 153.67 81.28 0) (unit 1)
+    (in_bom yes) (on_board yes) (dnp no) (fields_autoplaced)
+    (property "Reference" "TP2" (at 156.21 76.708 0)
+      (effects (font (size 1.27 1.27)) (justify left))
+    )
+    (property "Value" "TP-3V3" (at 156.21 79.248 0)
+      (effects (font (size 1.27 1.27)) (justify left))
+    )
+    (property "Footprint" "TestPoint:TestPoint_Pad_D1.0mm" (at 158.75 81.28 0)
+      (effects (font (size 1.27 1.27)) hide)
+    )
+    (property "Datasheet" "~" (at 158.75 81.28 0)
+      (effects (font (size 1.27 1.27)) hide)
+    )
+    (pin "1")
+    (instances
+      (project "isp32"
+        (path "/ca06a406-809a-4071-b112-487eee5c9315"
+          (reference "TP2") (unit 1)
+        )
+      )
+    )
+  )
   (symbol (lib_id "Device:LED_Small") (at 100.33 88.265 90) (unit 1)
     (in_bom yes) (on_board yes) (dnp no) (fields_autoplaced)
@@
       (effects (font (size 1.27 1.27)) (justify right))
     )
-    (property "Value" "1k" (at 340.995 50.8 0)
+    (property "Value" "10k" (at 340.995 50.8 0)
       (effects (font (size 1.27 1.27)) (justify right))
     )
@@
       (effects (font (size 1.27 1.27)) (justify right))
     )
-    (property "Value" "1k" (at 295.91 51.435 0)
+    (property "Value" "10k" (at 295.91 51.435 0)
       (effects (font (size 1.27 1.27)) (justify right))
     )
